File: pcb_hs/bakeneko-60-pcb.kicad_pcb (KiCad board)
At the start: 2 copper layers, 284.7 x 94.2 mm, 159 parts, among them J1 JST SH 4-pin, J2 AVR-ISP-6, SW1 Reset, U1 SRV05-4, U2 ATmega32U4-AU, Y1 16MHz

Commit message: Update bakeneko-60-pcb.kicad_pcb
Parts:
- moved D17 21.2 mm to (46.5, 29.6)
- moved D30 21.0 mm to (3.10, 48.5)
- moved D43 17.7 mm to (11.2, 68.0)
- moved D63 1.33 mm to (260.5, 87.0)
- moved D58 1.32 mm to (48.6, 87.0)
- moved D61 1.28 mm to (213.0, 87.0)
- moved D62 1.26 mm to (236.8, 87.0)
- moved D56 1.25 mm to (22.5, 87.0)
- moved D60 1.09 mm to (191.9, 87.0)
- moved D55 1.06 mm to (267.7, 68.0)
- moved D44 1.06 mm to (42.3, 68.0)
- moved D45 1.06 mm to (61.4, 68.0)
- moved D46 1.06 mm to (80.4, 68.0)
- moved D47 1.06 mm to (99.5, 68.0)
- moved D48 1.06 mm to (118.5, 68.0)
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Routing:
- net (no net): track 1207.3 -> 15.5 mm, vias 1 -> 0
- net COL10: track 394.5 -> 0.00 mm
- net COL6: track 333.4 -> 24.7 mm, vias 3 -> 2
- net COL13: track 254.9 -> 1.92 mm
- net COL11: track 199.8 -> 1.92 mm
- net COL9: track 165.5 -> 0.00 mm
- net COL7: track 128.2 -> 1.61 mm
- net COL3: track 117.2 -> 0.00 mm
- net COL0: track 100.5 -> 1.92 mm, vias 1 -> 0
- net COL5: track 91.2 -> 0.00 mm
- net ROW2: track 269.1 -> 204.0 mm, vias 2 -> 0
- net RST: track 88.7 -> 28.1 mm, vias 2 -> 1
- net ROW4: track 298.5 -> 238.0 mm, vias 2 -> 1
- net SCK: track 45.7 -> 0.00 mm, vias 2 -> 0
- net MOSI: track 45.6 -> 0.00 mm, vias 2 -> 0
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
Commit message: Update bakeneko-60-pcb.kicad_pcb
Parts:
- turned MX31 to 180 degrees
- turned MX32 to 180 degrees
